Commit message: updated paddle

File: src/final_project/urdf/sevenDOF.urdf (robot description, URDF)
Before this commit: robot sevenDOF, 36 links, 35 joints
Links:
- removed link cube
- removed link cube-xm
- removed link cube-xp
- removed link cube-ym
- removed link cube-yp
- removed link cube-zm
- removed link cube-zp
- added link paddle, mass 0.5; collision cylinder length=0.01 radius=0.15; visual cylinder length=0.01 radius=0.15
Joints:
- removed joint attach-cube
- removed joint attach-cube-xm
- removed joint attach-cube-xp
- removed joint attach-cube-ym
- removed joint attach-cube-yp
- removed joint attach-cube-zm
- removed joint attach-cube-zp
- added joint attach-paddle: type fixed, parent tip, child paddle

Commit message: Removed unnecessary definitions from URDF.

File: src/final_project/urdf/sevenDOF.urdf (robot description, URDF)
Before this commit: robot sevenDOF, 30 links, 29 joints
Links:
- removed link handbase
- removed link leftfinger
- removed link palm
- removed link rightfinger
Joints:
- removed joint attach-handbase
- removed joint attach-leftfinger
- removed joint attach-palm
- removed joint attach-rightfinger
